Commit message: gravcomp wip, added 4 joints

File: description/urdf/test_state_publisher.urdf.xacro (robot description, xacro)
@@ -27,4 +27,43 @@
     </visual>
   </link>
+  <link name="link_2">
+    <!-- <inertial>
+      <origin xyz="0 0 0" rpy="0 0 0"/>
+      <mass value="3.0"/>
+      <inertia ixx="0.001" ixy="0" ixz="0" iyy="0.001" iyz="0" izz="0.001"/>
+    </inertial> -->
+    <visual name="Cube">
+      <origin xyz="1 0 0" rpy="0 0 0"/>
+      <geometry>
+        <box size="0.24 0.14 0.22"/>
+      </geometry>
+    </visual>
+  </link>
+  <link name="link_3">
+    <!-- <inertial>
+      <origin xyz="0 0 0" rpy="0 0 0"/>
+      <mass value="3.0"/>
+      <inertia ixx="0.001" ixy="0" ixz="0" iyy="0.001" iyz="0" izz="0.001"/>
+    </inertial> -->
+    <visual name="Cube">
+      <origin xyz="1 0 0" rpy="0 0 0"/>
+      <geometry>
+        <box size="0.24 0.14 0.22"/>
+      </geometry>
+    </visual>
+  </link>
+  <link name="link_4">
+    <!-- <inertial>
+      <origin xyz="0 0 0" rpy="0 0 0"/>
+      <mass value="3.0"/>
+      <inertia ixx="0.001" ixy="0" ixz="0" iyy="0.001" iyz="0" izz="0.001"/>
+    </inertial> -->
+    <visual name="Cube">
+      <origin xyz="1 0 0" rpy="0 0 0"/>
+      <geometry>
+        <box size="0.24 0.14 0.22"/>
+      </geometry>
+    </visual>
+  </link>
   <joint name="joint_1" type="revolute">
     <origin xyz="0 -0.1 0" rpy="1.5708 1.5708 0"/>
@@ -32,4 +71,25 @@
     <child link="link_1"/>
     <axis xyz="0 0 1.0"/>
+    <limit lower="-1.39626" upper="-0.5236" effort="35.0" velocity="26.0"/>
+  </joint>
+  <joint name="joint_2" type="revolute">
+    <origin xyz="0 -0.1 0" rpy="1.5708 1.5708 0"/>
+    <parent link="link_1"/>
+    <child link="link_2"/>
+    <axis xyz="0 1.0 0"/>
+    <limit lower="-1.39626" upper="-0.5236" effort="35.0" velocity="26.0"/>
+  </joint>
+  <joint name="joint_3" type="revolute">
+    <origin xyz="0 -0.1 0" rpy="1.5708 1.5708 0"/>
+    <parent link="link_2"/>
+    <child link="link_3"/>
+    <axis xyz="0 1.0 0"/>
+    <limit lower="-1.39626" upper="-0.5236" effort="35.0" velocity="26.0"/>
+  </joint>
+  <joint name="joint_4" type="revolute">
+    <origin xyz="0 -0.1 0" rpy="1.5708 1.5708 0"/>
+    <parent link="link_3"/>
+    <child link="link_4"/>
+    <axis xyz="0 1.0 0"/>
     <limit lower="-1.39626" upper="-0.5236" effort="35.0" velocity="26.0"/>
   </joint>
@@ -44,9 +104,9 @@
           <param name="axis_direction">-1</param>
           <param name="position_offset">0.0</param>
-          <param name="gear_ratio">1.0</param>
+          <param name="gear_ratio">0.306569</param>
           <param name="torque_constant">0.09729</param>
           <param name="power_max">100.0</param>
-          <param name="position_min">-3.1415</param>
-          <param name="position_max">3.1415</param>
+          <param name="position_min">-9.5</param>
+          <param name="position_max">9.5</param>
           <param name="velocity_max">3.1415</param>
           <param name="soft_start_duration_ms">0</param>
@@ -58,16 +118,16 @@
           <state_interface name="effort"/>
       </joint>
-      <!-- <joint name="joint_2">
-          <param name="can_protocol">odrive</param>
+      <joint name="joint_2">
+          <param name="can_protocol">moteus</param>
           <param name="can_id">2</param>
           <param name="can_channel">1</param>
           <param name="axis_direction">-1</param>
           <param name="position_offset">0.0</param>
-          <param name="gear_ratio">1.0</param>
+          <param name="gear_ratio">0.2</param>
           <param name="torque_constant">0.09729</param>
-          <param name="effort_max">1.0</param>
-          <param name="position_min">-1.0</param>
-          <param name="position_max">1.0</param>
-          <param name="velocity_max">1.0</param>
+          <param name="power_max">100.0</param>
+          <param name="position_min">-9.5</param>
+          <param name="position_max">9.5</param>
+          <param name="velocity_max">3.1415</param>
           <param name="kp_max">1.0</param>
           <param name="kd_max">1.0</param>
@@ -85,15 +145,15 @@
       </joint>
       <joint name="joint_3">
-          <param name="can_protocol">odrive</param>
+          <param name="can_protocol">moteus</param>
           <param name="can_id">3</param>
           <param name="can_channel">1</param>
           <param name="axis_direction">-1</param>
           <param name="position_offset">0.0</param>
-          <param name="gear_ratio">1.0</param>
+          <param name="gear_ratio">0.2</param>
           <param name="torque_constant">0.09729</param>
-          <param name="effort_max">1.0</param>
-          <param name="position_min">-1.0</param>
-          <param name="position_max">1.0</param>
-          <param name="velocity_max">1.0</param>
+          <param name="power_max">100.0</param>
+          <param name="position_min">-11.3</param>
+          <param name="position_max">11.3</param>
+          <param name="velocity_max">3.1415</param>
           <param name="kp_max">1.0</param>
           <param name="kd_max">1.0</param>
@@ -109,5 +169,31 @@
           <state_interface name="velocity"/>
           <state_interface name="effort"/>
-      </joint> -->
+      </joint>
+      <joint name="joint_4">
+          <param name="can_protocol">moteus</param>
+          <param name="can_id">4</param>
+          <param name="can_channel">1</param>
+          <param name="axis_direction">-1</param>
+          <param name="position_offset">0.0</param>
+          <param name="gear_ratio">0.2</param>
+          <param name="torque_constant">0.09729</param>
+          <param name="power_max">100.0</param>
+          <param name="position_min">-12.5</param>
+          <param name="position_max">12.5</param>
+          <param name="velocity_max">3.1415</param>
+          <param name="kp_max">1.0</param>
+          <param name="kd_max">1.0</param>
+          <param name="ki_max">1.0</param>
+          <param name="soft_start_duration_ms">0</param>
+          <command_interface name="position"/>
+          <command_interface name="velocity"/>
+          <command_interface name="effort"/>
+          <command_interface name="kp"/>
+          <command_interface name="kd"/>
+          <command_interface name="ki"/>
+          <state_interface name="position"/>
+          <state_interface name="velocity"/>
+          <state_interface name="effort"/>
+      </joint>
   </ros2_control>
 </robot>

Commit message: gravcomp working so far, needs tuning

File: description/urdf/test_state_publisher.urdf.xacro (robot description, xacro)
@@ -124,5 +124,5 @@
           <param name="axis_direction">-1</param>
           <param name="position_offset">0.0</param>
-          <param name="gear_ratio">0.2</param>
+          <param name="gear_ratio">0.25</param>
           <param name="torque_constant">0.09729</param>
           <param name="power_max">100.0</param>
@@ -144,5 +144,5 @@
           <state_interface name="effort"/>
       </joint>
-      <joint name="joint_3">
+     <joint name="joint_3">
           <param name="can_protocol">moteus</param>
           <param name="can_id">3</param>
@@ -150,5 +150,5 @@
           <param name="axis_direction">-1</param>
           <param name="position_offset">0.0</param>
-          <param name="gear_ratio">0.2</param>
+          <param name="gear_ratio">0.25</param>
           <param name="torque_constant">0.09729</param>
           <param name="power_max">100.0</param>
@@ -176,5 +176,5 @@
           <param name="axis_direction">-1</param>
           <param name="position_offset">0.0</param>
-          <param name="gear_ratio">0.2</param>
+          <param name="gear_ratio">0.25</param>
           <param name="torque_constant">0.09729</param>
           <param name="power_max">100.0</param>

Commit message: update urdf with correct robot model

File: description/urdf/test_state_publisher.urdf.xacro (robot description, xacro)
@@ -1,96 +1,107 @@
 <?xml version="1.0"?>
 <robot xmlns:xacro="http://www.ros.org/wiki/xacro" name="test_state_publisher_robot">
-  <link name="base_link">
-    <!-- <inertial>
-      <origin xyz="0 0 0" rpy="0 0 0"/>
-      <mass value="3.0"/>
-      <inertia ixx="0.001" ixy="0" ixz="0" iyy="0.001" iyz="0" izz="0.001"/>
-    </inertial> -->
-    <visual name="Cube">
-      <origin xyz="0 0 0" rpy="0 0 0"/>
-      <geometry>
-        <box size="0.24 0.14 0.22"/>
-      </geometry>
-    </visual>
-  </link>
-  <link name="link_1">
-    <!-- <inertial>
-      <origin xyz="0 0 0" rpy="0 0 0"/>
-      <mass value="3.0"/>
-      <inertia ixx="0.001" ixy="0" ixz="0" iyy="0.001" iyz="0" izz="0.001"/>
-    </inertial> -->
-    <visual name="Cube">
-      <origin xyz="0 0 0" rpy="0 0 0"/>
-      <geometry>
-        <box size="0.24 0.14 0.22"/>
-      </geometry>
-    </visual>
-  </link>
-  <link name="link_2">
-    <!-- <inertial>
-      <origin xyz="0 0 0" rpy="0 0 0"/>
-      <mass value="3.0"/>
-      <inertia ixx="0.001" ixy="0" ixz="0" iyy="0.001" iyz="0" izz="0.001"/>
-    </inertial> -->
-    <visual name="Cube">
-      <origin xyz="1 0 0" rpy="0 0 0"/>
-      <geometry>
-        <box size="0.24 0.14 0.22"/>
-      </geometry>
-    </visual>
-  </link>
-  <link name="link_3">
-    <!-- <inertial>
-      <origin xyz="0 0 0" rpy="0 0 0"/>
-      <mass value="3.0"/>
-      <inertia ixx="0.001" ixy="0" ixz="0" iyy="0.001" iyz="0" izz="0.001"/>
-    </inertial> -->
-    <visual name="Cube">
-      <origin xyz="1 0 0" rpy="0 0 0"/>
-      <geometry>
-        <box size="0.24 0.14 0.22"/>
-      </geometry>
-    </visual>
-  </link>
-  <link name="link_4">
-    <!-- <inertial>
-      <origin xyz="0 0 0" rpy="0 0 0"/>
-      <mass value="3.0"/>
-      <inertia ixx="0.001" ixy="0" ixz="0" iyy="0.001" iyz="0" izz="0.001"/>
-    </inertial> -->
-    <visual name="Cube">
-      <origin xyz="1 0 0" rpy="0 0 0"/>
-      <geometry>
-        <box size="0.24 0.14 0.22"/>
-      </geometry>
-    </visual>
-  </link>
-  <joint name="joint_1" type="revolute">
-    <origin xyz="0 -0.1 0" rpy="1.5708 1.5708 0"/>
+  <link name="link1">
+    <inertial>
+      <origin xyz="0.005025224974257385 0.000591246956100272 0.1406485292017584" rpy="0 0 0"/>
+      <mass value="22.70774043141286"/>
+      <inertia ixx="0.138286" iyy="0.141753" izz="0.061066" ixy="-0.00012" iyz="-0.000635" ixz="-0.01416"/>
+    </inertial>
+    <visual>
+      <origin xyz="-0.05 -0.095 -0.0515" rpy="0 0 0"/>
+      <geometry>
+        <mesh filename="file://$(find moteus_control)/meshes/link1_1.stl" scale="0.001 0.001 0.001"/>
+      </geometry>
+      <material name="silver"/>
+    </visual>
+    <collision>
+      <origin xyz="-0.05 -0.095 -0.0515" rpy="0 0 0"/>
+      <geometry>
+        <mesh filename="file://$(find moteus_control)/meshes/link1_1.stl" scale="0.001 0.001 0.001"/>
+      </geometry>
+    </collision>
+  </link>
+  <link name="link2">
+    <inertial>
+      <origin xyz="0.0331249282490404 -0.008782165245542081 7.776382659974157e-05" rpy="0 0 0"/>
+      <mass value="4.469585742928346"/>
+      <inertia ixx="0.096735" iyy="0.00942" izz="0.097633" ixy="-0.0074" iyz="-5.6e-05" ixz="-8e-06"/>
+    </inertial>
+    <visual>
+      <origin xyz="-0.129452 -0.096 -0.258548" rpy="0 0 0"/>
+      <geometry>
+        <mesh filename="file://$(find moteus_control)/meshes/link2_1.stl" scale="0.001 0.001 0.001"/>
+      </geometry>
+      <material name="silver"/>
+    </visual>
+    <collision>
+      <origin xyz="-0.129452 -0.096 -0.258548" rpy="0 0 0"/>
+      <geometry>
+        <mesh filename="file://$(find moteus_control)/meshes/link2_1.stl" scale="0.001 0.001 0.001"/>
+      </geometry>
+    </collision>
+  </link>
+  <link name="link3">
+    <inertial>
+      <origin xyz="-0.014018350116589001 -0.04260563451756741 -1.5875033888224088e-05" rpy="0 0 0"/>
+      <mass value="1.8887513349591307"/>
+      <inertia ixx="0.01281" iyy="0.002988" izz="0.014892" ixy="-0.002317" iyz="-1e-06" ixz="-1e-06"/>
+    </inertial>
+    <visual>
+      <origin xyz="-0.164451 0.204 -0.258548" rpy="0 0 0"/>
+      <geometry>
+        <mesh filename="file://$(find moteus_control)/meshes/link3_1.stl" scale="0.001 0.001 0.001"/>
+      </geometry>
+      <material name="silver"/>
+    </visual>
+    <collision>
+      <origin xyz="-0.164451 0.204 -0.258548" rpy="0 0 0"/>
+      <geometry>
+        <mesh filename="file://$(find moteus_control)/meshes/link3_1.stl" scale="0.001 0.001 0.001"/>
+      </geometry>
+    </collision>
+  </link>
+  <link name="link4">
+    <inertial>
+      <origin xyz="-0.02856503032037011 -0.060805161547451636 -0.004181738483013175" rpy="0 0 0"/>
+      <mass value="1.4283524207710583"/>
+      <inertia ixx="0.003284" iyy="0.001129" izz="0.003752" ixy="-0.000246" iyz="-9.1e-05" ixz="3e-06"/>
+    </inertial>
+    <visual>
+      <origin xyz="-0.141217 0.404 -0.258515" rpy="0 0 0"/>
+      <geometry>
+        <mesh filename="file://$(find moteus_control)/meshes/link4_1.stl" scale="0.001 0.001 0.001"/>
+      </geometry>
+      <material name="silver"/>
+    </visual>
+    <collision>
+      <origin xyz="-0.141217 0.404 -0.258515" rpy="0 0 0"/>
+      <geometry>
+        <mesh filename="file://$(find moteus_control)/meshes/link4_1.stl" scale="0.001 0.001 0.001"/>
+      </geometry>
+    </collision>
+  </link>
+  <joint name="Joint1" type="revolute">
+    <origin xyz="0.05 0.095 0.0515" rpy="0 0 0"/>
     <parent link="base_link"/>
-    <child link="link_1"/>
-    <axis xyz="0 0 1.0"/>
-    <limit lower="-1.39626" upper="-0.5236" effort="35.0" velocity="26.0"/>
-  </joint>
-  <joint name="joint_2" type="revolute">
-    <origin xyz="0 -0.1 0" rpy="1.5708 1.5708 0"/>
-    <parent link="link_1"/>
-    <child link="link_2"/>
-    <axis xyz="0 1.0 0"/>
-    <limit lower="-1.39626" upper="-0.5236" effort="35.0" velocity="26.0"/>
-  </joint>
-  <joint name="joint_3" type="revolute">
-    <origin xyz="0 -0.1 0" rpy="1.5708 1.5708 0"/>
-    <parent link="link_2"/>
-    <child link="link_3"/>
-    <axis xyz="0 1.0 0"/>
-    <limit lower="-1.39626" upper="-0.5236" effort="35.0" velocity="26.0"/>
-  </joint>
-  <joint name="joint_4" type="revolute">
-    <origin xyz="0 -0.1 0" rpy="1.5708 1.5708 0"/>
-    <parent link="link_3"/>
-    <child link="link_4"/>
-    <axis xyz="0 1.0 0"/>
-    <limit lower="-1.39626" upper="-0.5236" effort="35.0" velocity="26.0"/>
+    <child link="link1"/>
+    <axis xyz="-0.0 -0.0 -1.0"/>
+  </joint>
+  <joint name="joint2" type="revolute">
+    <origin xyz="0.079452 0.001 0.207048" rpy="0 0 0"/>
+    <parent link="link1"/>
+    <child link="link2"/>
+    <axis xyz="-1.0 0.0 -0.0"/>
+  </joint>
+  <joint name="joint3" type="revolute">
+    <origin xyz="0.034999 -0.3 0.0" rpy="0 0 0"/>
+    <parent link="link2"/>
+    <child link="link3"/>
+    <axis xyz="-1.0 0.0 -0.0"/>
+  </joint>
+  <joint name="joint4" type="revolute">
+    <origin xyz="-0.023234 -0.2 -3.3e-05" rpy="0 0 0"/>
+    <parent link="link3"/>
+    <child link="link4"/>
+    <axis xyz="-1.0 -0.0 0.0"/>
   </joint>
   <ros2_control name="moteus_hardware_interface" type="system">

Commit message: add missing base link update rviz config

File: description/urdf/test_state_publisher.urdf.xacro (robot description, xacro)
@@ -1,4 +1,21 @@
 <?xml version="1.0"?>
 <robot xmlns:xacro="http://www.ros.org/wiki/xacro" name="test_state_publisher_robot">
+<material name="silver">
+  <color rgba="0.700 0.700 0.700 1.000"/>
+</material>  <link name="base_link">
+    <visual>
+      <origin xyz="0 0 0" rpy="0 0 0"/>
+      <geometry>
+        <mesh filename="file://$(find moteus_control)/meshes/base_link.stl" scale="0.001 0.001 0.001"/>
+      </geometry>
+      <material name="silver"/>
+    </visual>
+    <collision>
+      <origin xyz="0 0 0" rpy="0 0 0"/>
+      <geometry>
+        <mesh filename="file://$(find moteus_control)/meshes/base_link.stl" scale="0.001 0.001 0.001"/>
+      </geometry>
+    </collision>
+  </link>
   <link name="link1">
     <inertial>
@@ -81,5 +98,5 @@
     </collision>
   </link>
-  <joint name="Joint1" type="revolute">
+  <joint name="joint_1" type="continuous">
     <origin xyz="0.05 0.095 0.0515" rpy="0 0 0"/>
     <parent link="base_link"/>
@@ -87,5 +104,5 @@
     <axis xyz="-0.0 -0.0 -1.0"/>
   </joint>
-  <joint name="joint2" type="revolute">
+  <joint name="joint_2" type="continuous">
     <origin xyz="0.079452 0.001 0.207048" rpy="0 0 0"/>
     <parent link="link1"/>
@@ -93,5 +110,5 @@
     <axis xyz="-1.0 0.0 -0.0"/>
   </joint>
-  <joint name="joint3" type="revolute">
+  <joint name="joint_3" type="continuous">
     <origin xyz="0.034999 -0.3 0.0" rpy="0 0 0"/>
     <parent link="link2"/>
@@ -99,5 +116,5 @@
     <axis xyz="-1.0 0.0 -0.0"/>
   </joint>
-  <joint name="joint4" type="revolute">
+  <joint name="joint_4" type="continuous">
     <origin xyz="-0.023234 -0.2 -3.3e-05" rpy="0 0 0"/>
     <parent link="link3"/>

Commit message: rviz visualisation working changed hardware interface to report joint positions correctly

File: description/urdf/test_state_publisher.urdf.xacro (robot description, xacro)
@@ -40,11 +40,11 @@
   <link name="link2">
     <inertial>
-      <origin xyz="0.0331249282490404 -0.008782165245542081 7.776382659974157e-05" rpy="0 0 0"/>
+      <origin xyz="-0.03312492824904028 -7.751694596296044e-05 0.008782412126177253" rpy="0 0 0"/>
       <mass value="4.469585742928346"/>
-      <inertia ixx="0.096735" iyy="0.00942" izz="0.097633" ixy="-0.0074" iyz="-5.6e-05" ixz="-8e-06"/>
-    </inertial>
-    <visual>
-      <origin xyz="-0.129452 -0.096 -0.258548" rpy="0 0 0"/>
-      <geometry>
+      <inertia ixx="0.096735" iyy="0.097633" izz="0.00942" ixy="-8e-06" iyz="-5.6e-05" ixz="-0.0074"/>
+    </inertial>
+    <visual>
+    <origin xyz="0.029452 -0.094 -0.258548" rpy="0 0 0"/>
+    <geometry>
         <mesh filename="file://$(find moteus_control)/meshes/link2_1.stl" scale="0.001 0.001 0.001"/>
       </geometry>
@@ -52,5 +52,5 @@
     </visual>
     <collision>
-      <origin xyz="-0.129452 -0.096 -0.258548" rpy="0 0 0"/>
+      <origin xyz="0.029452 -0.094 -0.258548" rpy="0 0 0"/>
       <geometry>
         <mesh filename="file://$(find moteus_control)/meshes/link2_1.stl" scale="0.001 0.001 0.001"/>
@@ -60,10 +60,10 @@
   <link name="link3">
     <inertial>
-      <origin xyz="-0.014018350116589001 -0.04260563451756741 -1.5875033888224088e-05" rpy="0 0 0"/>
+      <origin xyz="0.014018350116598403 1.6121914526170955e-05 0.04260588139820243" rpy="0 0 0"/>
       <mass value="1.8887513349591307"/>
-      <inertia ixx="0.01281" iyy="0.002988" izz="0.014892" ixy="-0.002317" iyz="-1e-06" ixz="-1e-06"/>
-    </inertial>
-    <visual>
-      <origin xyz="-0.164451 0.204 -0.258548" rpy="0 0 0"/>
+      <inertia ixx="0.01281" iyy="0.014892" izz="0.002988" ixy="-1e-06" iyz="-1e-06" ixz="-0.002317"/>
+    </inertial>
+    <visual>
+      <origin xyz="0.064451 -0.094 -0.558548" rpy="0 0 0"/>
       <geometry>
         <mesh filename="file://$(find moteus_control)/meshes/link3_1.stl" scale="0.001 0.001 0.001"/>
@@ -72,5 +72,5 @@
     </visual>
     <collision>
-      <origin xyz="-0.164451 0.204 -0.258548" rpy="0 0 0"/>
+      <origin xyz="0.064451 -0.094 -0.558548" rpy="0 0 0"/>
       <geometry>
         <mesh filename="file://$(find moteus_control)/meshes/link3_1.stl" scale="0.001 0.001 0.001"/>
@@ -80,10 +80,10 @@
   <link name="link4">
     <inertial>
-      <origin xyz="-0.02856503032037011 -0.060805161547451636 -0.004181738483013175" rpy="0 0 0"/>
+      <origin xyz="0.02856503032038614 0.004181985363651317 0.06080540842808546" rpy="0 0 0"/>
       <mass value="1.4283524207710583"/>
-      <inertia ixx="0.003284" iyy="0.001129" izz="0.003752" ixy="-0.000246" iyz="-9.1e-05" ixz="3e-06"/>
-    </inertial>
-    <visual>
-      <origin xyz="-0.141217 0.404 -0.258515" rpy="0 0 0"/>
+      <inertia ixx="0.003284" iyy="0.003752" izz="0.001129" ixy="3e-06" iyz="-9.1e-05" ixz="-0.000246"/>
+    </inertial>
+    <visual>
+      <origin xyz="0.041217 -0.094033 -0.758548" rpy="0 0 0"/>
       <geometry>
         <mesh filename="file://$(find moteus_control)/meshes/link4_1.stl" scale="0.001 0.001 0.001"/>
@@ -92,5 +92,5 @@
     </visual>
     <collision>
-      <origin xyz="-0.141217 0.404 -0.258515" rpy="0 0 0"/>
+      <origin xyz="0.041217 -0.094033 -0.758548" rpy="0 0 0"/>
       <geometry>
         <mesh filename="file://$(find moteus_control)/meshes/link4_1.stl" scale="0.001 0.001 0.001"/>
@@ -105,20 +105,20 @@
   </joint>
   <joint name="joint_2" type="continuous">
-    <origin xyz="0.079452 0.001 0.207048" rpy="0 0 0"/>
+    <origin xyz="-0.079452 -0.001 0.207048" rpy="0 0 0"/>
     <parent link="link1"/>
     <child link="link2"/>
-    <axis xyz="-1.0 0.0 -0.0"/>
+    <axis xyz="1.0 -0.0 -0.0"/>
   </joint>
   <joint name="joint_3" type="continuous">
-    <origin xyz="0.034999 -0.3 0.0" rpy="0 0 0"/>
+    <origin xyz="-0.034999 0.0 0.3" rpy="0 0 0"/>
     <parent link="link2"/>
     <child link="link3"/>
-    <axis xyz="-1.0 0.0 -0.0"/>
+    <axis xyz="1.0 0.0 -0.0"/>
   </joint>
   <joint name="joint_4" type="continuous">
-    <origin xyz="-0.023234 -0.2 -3.3e-05" rpy="0 0 0"/>
+    <origin xyz="0.023234 3.3e-05 0.2" rpy="0 0 0"/>
     <parent link="link3"/>
     <child link="link4"/>
-    <axis xyz="-1.0 -0.0 0.0"/>
+    <axis xyz="1.0 -0.0 -0.0"/>
   </joint>
   <ros2_control name="moteus_hardware_interface" type="system">
@@ -204,5 +204,5 @@
           <param name="axis_direction">-1</param>
           <param name="position_offset">0.0</param>
-          <param name="gear_ratio">0.25</param>
+          <param name="gear_ratio">-0.25</param>
           <param name="torque_constant">0.09729</param>
           <param name="power_max">100.0</param>
